File: amp/amp.kicad_pcb (KiCad board)
At the start: 4 copper layers, 85.9 x 164.8 mm, 235 parts, among them J1 1017503, J2 1017503, J3 AudioJack3, J4 AudioJack3, J5 1017503, J6 1017503, K1 24V 10A NO, Q1 EPC2106, Q2 EPC2106, U1 TLV3201, U10 MAX15462, U11 R1283x, U12 LT1394, U13 LT1394, U14 LM5113SDX/NOPB, U15 LM5113SDX/NOPB, U16 74LVC2G14GV, U17 74LVC2G14GV, U2 LM4562, U3 TLV3541, U4 LM4562, U5 LM4562, U6 LM4562, U7 LM4562, U8 LM4562, U9 TLV3541

Commit message: shipped rev0 hardware
Parts:
- removed the C73 at (221.1, 266.9)
- removed the C74 at (221.1, 268.9)
- removed TP23, TP24, TP25, TP26: TestPoint, TestPoint:TestPoint_Pad_D1.0mm
- added ?: , , F.Cu at (167.0, 229.3)
- added ?: , , F.Cu at (177.9, 279.9)
- added ?: , , F.Cu at (223.8, 261.3)
- added ?: , , F.Cu at (206.7, 237.3)
- added ?: , , F.Cu at (208.8, 278.3)
- added ?: , , F.Cu at (234.5, 269.5)
- added ?: , , F.Cu at (190.3, 274.0)
- added ?: , , F.Cu at (177.9, 284.0)
- added ?: , , F.Cu at (184.9, 234.7)
- added ?: , , F.Cu at (192.8, 245.6)
- added ?: , , F.Cu at (202.9, 269.1)
- added ?: , , F.Cu at (187.4, 258.4)
- added ?: , , F.Cu at (175.8, 286.1)
- added ?: , , F.Cu at (213.2, 239.0)
- added ?: , , F.Cu at (219.5, 252.9)
- added ?: , , F.Cu at (189.6, 257.2)
- added ?: , , F.Cu at (200.7, 253.4)
- added ?: , , F.Cu at (216.2, 254.0)
- added ?: , , F.Cu at (192.8, 243.4)
- added ?: , , F.Cu at (218.2, 260.7)
- added ?: , , F.Cu at (225.4, 257.7)
- added ?: , , F.Cu at (196.8, 262.9)
- added ?: , , F.Cu at (221.7, 219.7)
- added ?: , , F.Cu at (210.2, 269.1)
- added ?: , , F.Cu at (222.5, 273.7)
- added ?: , , F.Cu at (213.2, 241.3)
- added ?: , , F.Cu at (178.0, 269.7)
- added ?: , , F.Cu at (186.0, 241.2)
- added ?: , , F.Cu at (206.8, 249.8)
- added ?: , , F.Cu at (225.3, 165.6)
- added ?: , , F.Cu at (189.4, 265.6)
- added ?: , , F.Cu at (203.6, 237.3)
- added ?: , , F.Cu at (229.0, 219.7)
- added ?: , , F.Cu at (213.9, 165.6)
- added ?: , , F.Cu at (211.1, 283.5)
- added C76: .1uF, Capacitor_SMD:C_0603_1608Metric, F.Cu at (214.6, 173.3)
- added C77: .1uF, Capacitor_SMD:C_0603_1608Metric, F.Cu at (181.0, 217.2)
- added C83: .1uF, Capacitor_SMD:C_0603_1608Metric, F.Cu at (214.6, 182.4)
- added C84: .1uF, Capacitor_SMD:C_0603_1608Metric, F.Cu at (223.4, 196.9)
- added C85: .1uF, Capacitor_SMD:C_0603_1608Metric, F.Cu at (172.0, 226.2)
- added C86: .1uF, Capacitor_SMD:C_0603_1608Metric, F.Cu at (221.1, 231.0)
- added C87: .1uF, Capacitor_SMD:C_0402_1005Metric, F.Cu at (204.8, 246.6)
- added C88: .1uF, Capacitor_SMD:C_0402_1005Metric, F.Cu at (196.9, 240.7)
- added R79: 0, Resistor_SMD:R_0603_1608Metric, F.Cu at (163.4, 222.2)
- added R80: 0, Resistor_SMD:R_0603_1608Metric, F.Cu at (221.3, 166.3)
- added R81: 0, Resistor_SMD:R_0603_1608Metric, F.Cu at (225.6, 180.8)
- added R82: 0, Resistor_SMD:R_0603_1608Metric, F.Cu at (214.5, 191.4)
- added R83: 0, Resistor_SMD:R_0603_1608Metric, F.Cu at (227.2, 222.0)
- added R84: 0, Resistor_SMD:R_0603_1608Metric, F.Cu at (187.8, 224.5)
- added REF**: TestPoint_THTPad_D1.0mm_Drill0.5mm, TestPoint:TestPoint_THTPad_D1.0mm_Drill0.5mm, F.Cu at (210.5, 261.7)
- added REF**: TestPoint_THTPad_D1.0mm_Drill0.5mm, TestPoint:TestPoint_THTPad_D1.0mm_Drill0.5mm, F.Cu at (203.6, 237.3)
- added REF**: TestPoint_THTPad_D1.0mm_Drill0.5mm, TestPoint:TestPoint_THTPad_D1.0mm_Drill0.5mm, F.Cu at (200.7, 253.4)
- added REF**: TestPoint_THTPad_D1.0mm_Drill0.5mm, TestPoint:TestPoint_THTPad_D1.0mm_Drill0.5mm, F.Cu at (190.3, 274.0)
- added REF**: TestPoint_THTPad_D1.0mm_Drill0.5mm, TestPoint:TestPoint_THTPad_D1.0mm_Drill0.5mm, F.Cu at (221.7, 219.7)
- added REF**: TestPoint_THTPad_D1.0mm_Drill0.5mm, TestPoint:TestPoint_THTPad_D1.0mm_Drill0.5mm, F.Cu at (189.4, 265.6)
- added REF**: TestPoint_THTPad_D1.0mm_Drill0.5mm, TestPoint:TestPoint_THTPad_D1.0mm_Drill0.5mm, F.Cu at (192.8, 243.4)
- added REF**: TestPoint_THTPad_D1.0mm_Drill0.5mm, TestPoint:TestPoint_THTPad_D1.0mm_Drill0.5mm, F.Cu at (177.9, 284.0)
- added REF**: TestPoint_THTPad_D1.0mm_Drill0.5mm, TestPoint:TestPoint_THTPad_D1.0mm_Drill0.5mm, F.Cu at (187.4, 258.4)
- added REF**: TestPoint_THTPad_D1.0mm_Drill0.5mm, TestPoint:TestPoint_THTPad_D1.0mm_Drill0.5mm, F.Cu at (229.0, 219.7)
- added REF**: TestPoint_THTPad_D1.0mm_Drill0.5mm, TestPoint:TestPoint_THTPad_D1.0mm_Drill0.5mm, F.Cu at (218.2, 260.7)
- added REF**: TestPoint_THTPad_D1.0mm_Drill0.5mm, TestPoint:TestPoint_THTPad_D1.0mm_Drill0.5mm, F.Cu at (234.5, 269.5)
- added REF**: TestPoint_THTPad_D1.0mm_Drill0.5mm, TestPoint:TestPoint_THTPad_D1.0mm_Drill0.5mm, F.Cu at (202.9, 269.1)
- added REF**: TestPoint_THTPad_D1.0mm_Drill0.5mm, TestPoint:TestPoint_THTPad_D1.0mm_Drill0.5mm, F.Cu at (175.8, 286.1)
- added REF**: TestPoint_THTPad_D1.0mm_Drill0.5mm, TestPoint:TestPoint_THTPad_D1.0mm_Drill0.5mm, F.Cu at (206.8, 249.8)
- added REF**: TestPoint_THTPad_D1.0mm_Drill0.5mm, TestPoint:TestPoint_THTPad_D1.0mm_Drill0.5mm, F.Cu at (177.9, 279.9)
- added REF**: TestPoint_THTPad_D1.0mm_Drill0.5mm, TestPoint:TestPoint_THTPad_D1.0mm_Drill0.5mm, F.Cu at (225.4, 257.7)
- added REF**: TestPoint_THTPad_D1.0mm_Drill0.5mm, TestPoint:TestPoint_THTPad_D1.0mm_Drill0.5mm, F.Cu at (225.3, 165.6)
- added REF**: TestPoint_THTPad_D1.0mm_Drill0.5mm, TestPoint:TestPoint_THTPad_D1.0mm_Drill0.5mm, F.Cu at (178.0, 269.7)
- added REF**: TestPoint_THTPad_D1.0mm_Drill0.5mm, TestPoint:TestPoint_THTPad_D1.0mm_Drill0.5mm, F.Cu at (211.1, 283.5)
- added REF**: TestPoint_THTPad_D1.0mm_Drill0.5mm, TestPoint:TestPoint_THTPad_D1.0mm_Drill0.5mm, F.Cu at (219.5, 252.9)
- added REF**: TestPoint_THTPad_D1.0mm_Drill0.5mm, TestPoint:TestPoint_THTPad_D1.0mm_Drill0.5mm, F.Cu at (223.8, 261.3)
- added REF**: TestPoint_THTPad_D1.0mm_Drill0.5mm, TestPoint:TestPoint_THTPad_D1.0mm_Drill0.5mm, F.Cu at (213.9, 165.6)
- added REF**: TestPoint_THTPad_D1.0mm_Drill0.5mm, TestPoint:TestPoint_THTPad_D1.0mm_Drill0.5mm, F.Cu at (206.7, 237.3)
- added REF**: TestPoint_THTPad_D1.0mm_Drill0.5mm, TestPoint:TestPoint_THTPad_D1.0mm_Drill0.5mm, F.Cu at (196.8, 262.9)
- added REF**: TestPoint_THTPad_D1.0mm_Drill0.5mm, TestPoint:TestPoint_THTPad_D1.0mm_Drill0.5mm, F.Cu at (189.6, 257.2)
- added REF**: TestPoint_THTPad_D1.0mm_Drill0.5mm, TestPoint:TestPoint_THTPad_D1.0mm_Drill0.5mm, F.Cu at (216.2, 254.0)
- added REF**: TestPoint_THTPad_D1.0mm_Drill0.5mm, TestPoint:TestPoint_THTPad_D1.0mm_Drill0.5mm, F.Cu at (213.2, 239.0)
- added REF**: TestPoint_THTPad_D1.0mm_Drill0.5mm, TestPoint:TestPoint_THTPad_D1.0mm_Drill0.5mm, F.Cu at (184.9, 234.7)
- added REF**: TestPoint_THTPad_D1.0mm_Drill0.5mm, TestPoint:TestPoint_THTPad_D1.0mm_Drill0.5mm, F.Cu at (186.0, 241.2)
- added REF**: TestPoint_THTPad_D1.0mm_Drill0.5mm, TestPoint:TestPoint_THTPad_D1.0mm_Drill0.5mm, F.Cu at (222.5, 273.7)
- added REF**: TestPoint_THTPad_D1.0mm_Drill0.5mm, TestPoint:TestPoint_THTPad_D1.0mm_Drill0.5mm, F.Cu at (210.2, 269.1)
- added REF**: TestPoint_THTPad_D1.0mm_Drill0.5mm, TestPoint:TestPoint_THTPad_D1.0mm_Drill0.5mm, F.Cu at (192.8, 245.6)
- added REF**: TestPoint_THTPad_D1.0mm_Drill0.5mm, TestPoint:TestPoint_THTPad_D1.0mm_Drill0.5mm, F.Cu at (213.2, 241.3)
- C11, C14, C16, C18, C19, C21: footprint Capacitor_SMD:C_0402_1005Metric -> Capacitor_SMD:C_0603_1608Metric
- C54, C69, C70, R73, R74: moved to B.Cu
- moved C54 88.5 mm to (223.0, 259.8)
- moved C69 86.1 mm to (220.6, 263.5), turned to 180 degrees
- moved R73 80.9 mm to (223.5, 257.7), turned to -90 degrees
- moved R74 79.4 mm to (217.5, 259.2), turned to -90 degrees
- moved C70 77.4 mm to (220.6, 261.5), turned to 180 degrees
- moved C68 76.1 mm to (221.5, 261.6), turned to -90 degrees
- moved R71 76.0 mm to (222.8, 262.3), turned to 90 degrees
- moved TP9 54.6 mm to (180.6, 284.0)
- moved TP15 47.5 mm to (175.8, 284.0), turned to 180 degrees
- moved TP16 38.3 mm to (175.8, 279.9), turned to 180 degrees
- moved C82 26.2 mm to (163.7, 238.0), turned to 90 degrees
- moved C33 22.1 mm to (165.7, 238.0), turned to 90 degrees
- moved C39 18.9 mm to (167.5, 237.4), turned to 90 degrees
- moved R49 18.1 mm to (185.2, 243.5), turned to -135 degrees
- moved C49 16.3 mm to (183.8, 236.8), turned to -135 degrees
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Connections:
- C11 pad 1: +5V6 -> Net-(C11-Pad1)
- C11 pad 2: -5V6 -> GND
- C14 pad 1: +5V6 -> Net-(C14-Pad1)
- C14 pad 2: -5V6 -> GND
- C16 pad 1: +5V6 -> Net-(C16-Pad1)
- C16 pad 2: -5V6 -> GND
- C18 pad 1: +5V6 -> Net-(C18-Pad1)
- C18 pad 2: -5V6 -> GND
- C19 pad 1: +5V6 -> Net-(C19-Pad1)
- C19 pad 2: -5V6 -> GND
- C21 pad 1: +5V6 -> Net-(C21-Pad1)
- C21 pad 2: -5V6 -> GND
- C56 pad 2: -5V6 -> GND
- C57 pad 2: -5V6 -> GND
- U1 pad 4: /V_BIAS_L -> GND
- U11 pad 13: (no net) -> GND
- U2 pad 8: +5V6 -> Net-(C19-Pad1)
- U4 pad 8: +5V6 -> Net-(C11-Pad1)
- U5 pad 8: +5V6 -> Net-(C14-Pad1)
- U6 pad 8: +5V6 -> Net-(C18-Pad1)
- U7 pad 8: +5V6 -> Net-(C21-Pad1)
- U8 pad 8: +5V6 -> Net-(C16-Pad1)
Routing:
- net GND: track 8.16 -> 221.5 mm, vias 2 -> 105
- net /V_BIAS_L: track 0.00 -> 150.1 mm, vias 0 -> 8
- net -5V6: track 0.00 -> 136.4 mm, vias 0 -> 13
- net +5V6: track 0.00 -> 135.4 mm, vias 0 -> 7
- net +24V: track 33.1 -> 126.3 mm, vias 3 -> 6
- net Net-(C42-Pad1): track 0.00 -> 76.5 mm
- net /VOL_ADJ_L: track 0.00 -> 66.1 mm, vias 0 -> 3
- net /VOL_ADJ_R: track 0.00 -> 50.1 mm, vias 0 -> 1
- net +5V: track 1.65 -> 48.1 mm, vias 2 -> 14
- net Net-(D1-Pad1): track 0.00 -> 42.1 mm, vias 0 -> 1
- net Net-(C50-Pad2): track 8.01 -> 49.4 mm
- net Net-(R11-Pad3): track 0.00 -> 40.3 mm, vias 0 -> 1
- net /EQ_ADJ_L: track 0.00 -> 39.5 mm, vias 0 -> 2
- net /EQ_ADJ_R: track 0.00 -> 38.8 mm, vias 0 -> 2
- net Net-(C51-Pad2): track 10.5 -> 49.0 mm, vias 0 -> 2
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- added copper zone on F.Cu, net +24V
- added copper zone on In2.Cu, net -5V6
- added copper zone on B.Cu, net /V_BIAS_R
- added copper zone on In1.Cu, net GND
- removed copper zone on B.Cu, net -5V6
- removed copper zone on F.Cu, net GND
Other:
- board text added: "+5V6"
- board text added: "-5V6"
- board text added: "Adi R"
- board text added: "GaN CLASS-D AMP"
- board text added: "SATURNS R COMING"
- board text added: "V0.0"
- board text removed: "666K triwavegen"
- board text removed: "GaN"
- board text removed: "bax EQ"
- board text removed: "bax vol ctrl"
- board text removed: "bias gen"
- board text removed: "buck"
- board text removed: "dc block & bias"
- board text removed: "deadtime gen"
- board text removed: "discrete modulation"
- board text removed: "gate drive stages"
- board text removed: "half bridge L"
- board text removed: "half bridge R"
- board text removed: "left bax"
- board text removed: "modulation"
- board text removed: "potentially flip"
- board text removed: "right bax"
- board text removed: "route traces in inner layers"
