File: amp/amp.kicad_sch (KiCad schematic)
At the start: 168 parts, among them J1 AudioPlug3, J2 AudioPlug3, Q1 EPC2106, Q2 EPC2106, U1 LM4562, U10 TLV3541, U11 LM4040DBZ-2.5, U12 LM5113SDX/NOPB, U13 LM5113SDX/NOPB, U14 LT1394, U15 LT1394, U2 LM4562, U3 LM4562, U4 LM4562, U5 LM4562, U6 LM4562, U7 TLV3201, U8 TLV3541, U9 MAX15462

Commit message: lots of schem and layouts updates
Parts:
- removed C12, C13, C19, C42, C43: 22uF, Capacitor_THT:CP_Radial_D5.0mm_P2.00mm, symbol Device:C_Polarized_Small_US
- removed C21, C38: 1uF, symbol Device:C_Small
- removed C22, C23: .1uF, symbol Device:C_Small
- removed J1, J2: AudioPlug3, symbol Connector:AudioPlug3
- removed R10, R5, R55, R56: 5K, symbol Device:R
- removed R11: 200, symbol Device:R
- removed R42, R43, R44, R45, R57, R58: 0, symbol Device:R
- removed TP13, TP17, TP27, TP4, TP5: TestPoint, symbol Connector:TestPoint
- removed U11: LM4040DBZ-2.5, Package_TO_SOT_SMD:SOT-23, symbol Reference_Voltage:LM4040DBZ-2.5
- added C2, C3, C81: 10uf, Capacitor_SMD:C_1206_3216Metric, symbol Device:C_Small
- added C25, C33, C4, C44, C5, C50, C51, C54, C55, C69, C70, C71, C73, C82: 10uf, Capacitor_SMD:C_0805_2012Metric, symbol Device:C_Small
- added C28, C80: .1uF, Capacitor_SMD:C_0402_1005Metric, symbol Device:C_Small
- added C34, C53, C68, C74: 1uF, Capacitor_SMD:C_0402_1005Metric, symbol Device:C_Small
- added C49: 22uF, Capacitor_SMD:C_0805_2012Metric, symbol Device:C_Small
- added C64, C65, C66, C67: 100pF, Capacitor_SMD:C_0805_2012Metric, symbol Device:C_Small
- added C7, C9: 1.5mF, Capacitor_THT:CP_Radial_D12.5mm_P5.00mm, symbol Device:C_Polarized_US
- added D1: BAT46WH, Diode_SMD:D_SOD-123F, symbol Diode:BAT46
- added D10, D11, D12, D13: RB551V, Package_TO_SOT_SMD:SOT-23, symbol lt1394:RB551V
- added D2, D3, D6, D7: LED, LED_SMD:LED_0805_2012Metric_Pad1.15x1.40mm_HandSolder, symbol Device:LED
- added D4, D5: 30V 800mA 200mV, Diode_SMD:D_SOD-323, symbol Diode:1N5818
- added FL1: 8A 700 Ohm 125V CMC, footprints:ECMS1V1306-701-R, symbol Device:Filter_EMI_CommonMode
- added J1, J2, J5, J6: 1017503, footprints:1017503, symbol Connector:Screw_Terminal_01x02
- added J3, J4: AudioJack3, footprints:SJ-3523-SMT, symbol Connector:AudioJack3
- added JP1: Jumper_2_Open, Connector_PinHeader_2.54mm:PinHeader_1x02_P2.54mm_Vertical, symbol Jumper:Jumper_2_Open
- added K1: 24V 10A NO, footprints:AZ9375-1A-24DEF, symbol Relay:ADW11
- added L1: 100uH 125mOhm 2.8A, Inductor_SMD:L_12x12mm_H8mm, symbol Device:L
- added L3, L4: 4.7uH, Inductor_SMD:L_0805_2012Metric_Pad1.15x1.40mm_HandSolder, symbol Device:L
- added L5, L6: 330nH, footprints:EXL1V0503-R33-R, symbol Device:L
- added R12, R69, R7, R70, R8: 10K, Resistor_SMD:R_0603_1608Metric, symbol Device:R
- added R13: 1K5, Resistor_SMD:R_0805_2012Metric, symbol Device:R
- added R23, R51, R52: 330, Resistor_SMD:R_0805_2012Metric, symbol Device:R
- added R3: 100 16W 1%, Resistor_SMD:R_2512_6332Metric, symbol Device:R
- added R38, R39: 2K, Resistor_SMD:R_0603_1608Metric, symbol Device:R
- added R40, R41: 46K4, Resistor_SMD:R_0603_1608Metric, symbol Device:R
- added R47, R48: 10K .1%, Resistor_SMD:R_0603_1608Metric, symbol Device:R
- added R49, R50: DNP, Resistor_SMD:R_0805_2012Metric, symbol Device:R
- added R6: 10K, Resistor_SMD:R_0805_2012Metric, symbol Device:R
- added R65, R66, R67, R68: 47, Resistor_SMD:R_0805_2012Metric, symbol Device:R
- added R71, R72, R73, R74, R75, R76: 0, Resistor_SMD:R_0402_1005Metric, symbol Device:R
- added R77, R78: 100K, Resistor_SMD:R_0805_2012Metric, symbol Device:R
- added TP15, TP8, TP9: TestPoint, TestPoint:TestPoint_Pad_2.5x2.5mm, symbol Connector:TestPoint
- added TP23: TestPoint, TestPoint:TestPoint_Pad_D1.0mm, symbol Connector:TestPoint
- added U11: R1283x, Package_DFN_QFN:DFN-12-1EP_3x3mm_P0.5mm_EP1.6x2.5mm, symbol lt1394:R1283K002C-TR
- added U16, U17: 74LVC2G14GV, Package_TO_SOT_SMD:SOT-363_SC-70-6, symbol lt1394:74LVC2G14GV
- C1: renamed from C9; footprint (none) -> Capacitor_SMD:C_0603_1608Metric
- C11: renamed from C54; footprint (none) -> Capacitor_SMD:C_0402_1005Metric
- C12: renamed from C17; footprint (none) -> Capacitor_SMD:C_0402_1005Metric
- C14: renamed from C55; footprint (none) -> Capacitor_SMD:C_0402_1005Metric
- C16: renamed from C56; footprint (none) -> Capacitor_SMD:C_0402_1005Metric
- C18: renamed from C57; footprint (none) -> Capacitor_SMD:C_0402_1005Metric
- C19: renamed from C58; footprint (none) -> Capacitor_SMD:C_0402_1005Metric
- C20: renamed from C1; footprint (none) -> Capacitor_SMD:C_1206_3216Metric; MPN (none) -> CL31A106MBHNNNE
- C21: renamed from C59; footprint (none) -> Capacitor_SMD:C_0402_1005Metric
- C22: renamed from C2; footprint (none) -> Capacitor_SMD:C_1206_3216Metric; MPN (none) -> CL31A106MBHNNNE
- C23: renamed from C3; footprint (none) -> Capacitor_SMD:C_1206_3216Metric; MPN (none) -> CL31A106MBHNNNE
- C24: renamed from C4; footprint (none) -> Capacitor_SMD:C_1206_3216Metric; MPN (none) -> CL31A106MBHNNNE
- C26: renamed from C5; footprint (none) -> Capacitor_SMD:C_1206_3216Metric; MPN (none) -> CL31A106MBHNNNE
- C27: renamed from C11; footprint (none) -> Capacitor_SMD:C_0402_1005Metric; MPN (none) -> CL21B105KBFNNNG
- C29: renamed from C14; footprint (none) -> Capacitor_SMD:C_0402_1005Metric; MPN (none) -> CL21B105KBFNNNG
- C30: renamed from C18; footprint (none) -> Capacitor_SMD:C_0805_2012Metric; MPN (none) -> CL31A106MBHNNNE
- C31: renamed from C28; footprint (none) -> Capacitor_SMD:C_0805_2012Metric
- C32: renamed from C29; footprint (none) -> Capacitor_SMD:C_0805_2012Metric
- C35: renamed from C30; footprint (none) -> Capacitor_SMD:C_0805_2012Metric
- C36: renamed from C31; footprint (none) -> Capacitor_SMD:C_0805_2012Metric
- C37: renamed from C34; footprint (none) -> Capacitor_SMD:C_0805_2012Metric
- C38: renamed from C35; footprint (none) -> Capacitor_SMD:C_0805_2012Metric
- C39: value 1uF -> .1uF; footprint (none) -> Capacitor_SMD:C_0402_1005Metric
- C40: value 10Uf -> 150pF; footprint (none) -> Capacitor_SMD:C_0603_1608Metric; MPN (none) -> CC0805KRX7R9BB151
- C41: value 10uf -> 150pF; footprint (none) -> Capacitor_SMD:C_0603_1608Metric; MPN (none) -> CC0805KRX7R9BB151
- C42: renamed from C36; footprint (none) -> Capacitor_SMD:C_0805_2012Metric
- C43: renamed from C37; footprint (none) -> Capacitor_SMD:C_0805_2012Metric
- C45: footprint (none) -> Capacitor_SMD:C_0805_2012Metric; MPN (none) -> CL31A106MBHNNNE
- C46: value 10Uf -> DNP; footprint (none) -> Capacitor_SMD:C_0805_2012Metric; MPN (none) -> CL21A226MAYNNNE
- C47: value 1uF -> DNP; footprint (none) -> Capacitor_SMD:C_0805_2012Metric; MPN (none) -> CL21A226MAYNNNE
- C48: value 1uF -> 22uF; footprint (none) -> Capacitor_SMD:C_0805_2012Metric; MPN (none) -> CL21A226MAYNNNE
- C52: renamed from C20; footprint (none) -> Capacitor_SMD:C_0402_1005Metric; MPN (none) -> CL21B105KBFNNNG
- C56: renamed from C50; footprint (none) -> Capacitor_SMD:C_0402_1005Metric
- C57: renamed from C51; footprint (none) -> Capacitor_SMD:C_0402_1005Metric
- C58: renamed from C24; footprint (none) -> Capacitor_SMD:C_0402_1005Metric; MPN (none) -> CML0805C0G220JT50V
- C59: renamed from C25; footprint (none) -> Capacitor_SMD:C_0402_1005Metric; MPN (none) -> CML0805C0G220JT50V
- C6: renamed from C15; footprint (none) -> Capacitor_SMD:C_0402_1005Metric
- C60: renamed from C26; footprint (none) -> Capacitor_SMD:C_0402_1005Metric; MPN (none) -> CML0805C0G220JT50V
- C61: renamed from C27; footprint (none) -> Capacitor_SMD:C_0402_1005Metric; MPN (none) -> CML0805C0G220JT50V
- C62: renamed from C32; footprint (none) -> Capacitor_SMD:C_0402_1005Metric
- C63: renamed from C33; footprint (none) -> Capacitor_SMD:C_0402_1005Metric
- C78: renamed from C53; footprint Capacitor_THT:CP_Radial_D7.5mm_P2.50mm -> Capacitor_THT:CP_Radial_D12.5mm_P5.00mm
- C79: renamed from C52; footprint Capacitor_THT:CP_Radial_D7.5mm_P2.50mm -> Capacitor_THT:CP_Radial_D12.5mm_P5.00mm
- C8: renamed from C16; footprint (none) -> Capacitor_SMD:C_0402_1005Metric
- L2: renamed from L1; footprint Inductor_SMD:L_10.4x10.4_H4.8 -> Inductor_SMD:L_Vishay_IHLP-1616; MPN (none) -> LQH44PH470MPRL
- Q1, Q2: footprint (none) -> footprints:epc2106
- R1, R2: footprint (none) -> Resistor_SMD:R_0603_1608Metric
- R10: renamed from R7; footprint (none) -> Resistor_SMD:R_0603_1608Metric
- R11: renamed from R9; footprint (none) -> footprints:PTA4544-2010CIB103
- R14, R15: footprint (none) -> Resistor_SMD:R_0805_2012Metric
- R16: renamed from R12; footprint (none) -> Resistor_SMD:R_0805_2012Metric
- R17: renamed from R13; footprint (none) -> Resistor_SMD:R_0805_2012Metric
- R18: renamed from R16; footprint (none) -> Resistor_SMD:R_0805_2012Metric
- R19: renamed from R17; footprint (none) -> Resistor_SMD:R_0805_2012Metric
- R20: renamed from R18; footprint (none) -> Resistor_SMD:R_0805_2012Metric
- R21: renamed from R19; footprint (none) -> Resistor_SMD:R_0805_2012Metric
- R22: renamed from R8; footprint (none) -> Resistor_SMD:R_0805_2012Metric
- R24: renamed from R26; footprint (none) -> Resistor_SMD:R_0805_2012Metric
- R25: renamed from R27; footprint (none) -> footprints:PTA4544-2010CIB103
- R26: renamed from R28; footprint (none) -> Resistor_SMD:R_0805_2012Metric
- R27: renamed from R29; footprint (none) -> Resistor_SMD:R_0805_2012Metric
- R28: renamed from R30; footprint (none) -> Resistor_SMD:R_0805_2012Metric
- R29: renamed from R31; footprint (none) -> Resistor_SMD:R_0805_2012Metric
- R30: renamed from R32; footprint (none) -> footprints:PTA4544-2010CIB103
- R31: renamed from R33; footprint (none) -> Resistor_SMD:R_0805_2012Metric
- R32: renamed from R34; footprint (none) -> Resistor_SMD:R_0805_2012Metric
- R33: renamed from R35; footprint (none) -> Resistor_SMD:R_0805_2012Metric
- R34: renamed from R40; footprint (none) -> Resistor_SMD:R_0805_2012Metric
- R35: renamed from R41; footprint (none) -> Resistor_SMD:R_0805_2012Metric
- R36: renamed from R46; footprint (none) -> Resistor_SMD:R_0805_2012Metric
- R37: renamed from R47; footprint (none) -> Resistor_SMD:R_0805_2012Metric
- R4: renamed from R3; footprint (none) -> Resistor_SMD:R_0603_1608Metric
- R42: renamed from R48; footprint (none) -> Resistor_SMD:R_0805_2012Metric
- R43: renamed from R49; footprint (none) -> footprints:PTA4544-2010CIB103
- R44: renamed from R50; footprint (none) -> Resistor_SMD:R_0805_2012Metric
- R45: renamed from R51; footprint (none) -> Resistor_SMD:R_0805_2012Metric
- R46: renamed from R52; footprint (none) -> Resistor_SMD:R_0805_2012Metric
- R5: renamed from R4; value 5K -> 10K; footprint (none) -> Resistor_SMD:R_0805_2012Metric
- R53, R54: value 0 -> 10K; footprint (none) -> Resistor_SMD:R_0805_2012Metric
- R55: renamed from R20; value R -> 1K; footprint (none) -> Resistor_SMD:R_0402_1005Metric
- R56: renamed from R21; footprint (none) -> Resistor_SMD:R_0402_1005Metric
- R57: renamed from R22; value R -> 1K; footprint (none) -> Resistor_SMD:R_0402_1005Metric
- R58: renamed from R23; footprint (none) -> Resistor_SMD:R_0402_1005Metric
- R59: renamed from R24; footprint (none) -> Resistor_SMD:R_0402_1005Metric
- R60: renamed from R25; footprint (none) -> Resistor_SMD:R_0402_1005Metric
- R61: renamed from R36; footprint (none) -> Resistor_SMD:R_0402_1005Metric
- R62: renamed from R37; footprint (none) -> Resistor_SMD:R_0402_1005Metric
- R63: renamed from R38; footprint (none) -> Resistor_SMD:R_0402_1005Metric
- R64: renamed from R39; footprint (none) -> Resistor_SMD:R_0402_1005Metric
- R9: renamed from R6; footprint (none) -> Resistor_SMD:R_0603_1608Metric
- TP1, TP10, TP24, TP25, TP26: footprint (none) -> TestPoint:TestPoint_Pad_D1.0mm
- TP11: renamed from TP12; footprint (none) -> TestPoint:TestPoint_Pad_D1.0mm
- TP12: renamed from TP14; footprint (none) -> TestPoint:TestPoint_Pad_D1.0mm
- TP13: renamed from TP15; footprint (none) -> TestPoint:TestPoint_Pad_D1.0mm
- TP14: renamed from TP11; footprint (none) -> TestPoint:TestPoint_Pad_2.5x2.5mm
- TP16, TP2, TP3: footprint (none) -> TestPoint:TestPoint_Pad_2.5x2.5mm
- TP17: renamed from TP18; footprint (none) -> TestPoint:TestPoint_Pad_D1.0mm
- TP18: renamed from TP19; footprint (none) -> TestPoint:TestPoint_Pad_D1.0mm
- TP19: renamed from TP20; footprint (none) -> TestPoint:TestPoint_Pad_D1.0mm
- TP20: renamed from TP21; footprint (none) -> TestPoint:TestPoint_Pad_D1.0mm
- TP21: renamed from TP22; footprint (none) -> TestPoint:TestPoint_Pad_D1.0mm
- TP22: renamed from TP23; footprint (none) -> TestPoint:TestPoint_Pad_D1.0mm
- TP4: renamed from TP6; footprint (none) -> TestPoint:TestPoint_Pad_D1.0mm
- TP5: renamed from TP7; footprint (none) -> TestPoint:TestPoint_Pad_D1.0mm
- TP6: renamed from TP8; footprint (none) -> TestPoint:TestPoint_Pad_2.5x2.5mm
- TP7: renamed from TP9; footprint (none) -> TestPoint:TestPoint_Pad_2.5x2.5mm
- U12: renamed from U14; footprint SO-8_S_LIT -> footprints:LT1394CS8-PBF
- U13: renamed from U15; footprint SO-8_S_LIT -> footprints:LT1394CS8-PBF
- U14: renamed from U12; footprint SDC10A -> footprints:LM5113SDX&slash_NOPB
- U15: renamed from U13; footprint SDC10A -> footprints:LM5113SDX&slash_NOPB
- renumbered C6 to C10, C7 to C13, C8 to C15, C10 to C17, C44 to C72, C49 to C75, D1 to D8, D2 to D9, L2 to L7, L3 to L8, U7 to U1, U9 to U10, U1 to U2, U8 to U3, U2 to U4, U3 to U5, U4 to U6, U5 to U7, U6 to U8, U10 to U9
Connections:
- net +2V5 is gone; now on net GND: U2.3 (+), U2.5 (+)
- net V_BIAS_L  is gone; now on net V_BIAS_L: U2.6 (-), U2.7
- net +24V: now also C3.1, C68.1, C69.1, C7.1, C70.1, C71.1, C73.1, C74.1, C81.1, C9.1, D2.2 (A), L1.2, TP8.1; no longer C39.1, C40.1, C41.1, C45.1, C46.1, C47.1
- net +5V: now also C28.2, C33.1, C34.1, C80.2, C82.1, D3.2 (A), J2.2 (Pin_2), L3.2, R69.2, R7.2, R71.1, R72.1, U11.11 (PVcc), U11.5 (CE), U11.8 (Vcc), U16.5, U17.5; no longer C11.1, C14.1, C16.1, C18.1, C19.1, C21.1, C52.1, C56.1, C57.1, D8.2 (A), D9.2 (A), TP2.1, U12.1 (V+), U13.1 (V+), U14.1 (VDD), U15.1 (VDD), U2.8 (V+), U4.8 (V+), U5.8 (V+), U6.8 (V+), U7.8 (V+), U8.8 (V+)
- net AUDIO_IN_L: now also C5.1, J3.T
- net AUDIO_IN_R: now also C4.1, J3.R
- net BUFFERED_L: now also U4.6 (-), U4.7; no longer U5.6 (-), U5.7
- net BUFFERED_R: now also U4.1, U4.2 (-); no longer U4.6 (-), U4.7
- net EQ_ADJ_L: now also U8.7, C51.1; no longer TP18.1, U13.2 (+), U8.1
- net EQ_ADJ_R: now also U8.1, C50.1; no longer TP16.1, TP17.1, U12.2 (+), U8.7
- net GH_L: now also R75.2
- net GH_R: now also R73.2
- net GL_L: now also R76.2
- net GL_R: now also R74.2
- net GND: now also C39.2, C47.2, C48.2, U10.5 (MODE), C2.2, C28.1, C3.2, C33.2, C34.2, C44.2, C49.2, C53.2, C54.1, C55.1, C64.2, C65.2, C66.2, C67.2, C68.2, C69.2, C7.2, C70.2, C71.2, C73.2, C74.2, C80.1, C81.2, C82.2, C9.2, D7.2 (A), FL1.4, J2.1 (Pin_1), J3.S, J4.S, J5.2 (Pin_2), J6.2 (Pin_2), JP1.2 (B), L4.1, R13.2, R23.2, R47.1, R51.2, R70.1, R77.1, R78.1, R8.1, TP9.1, U11.10 (GND), U11.12 (PGND), U16.2, U16.2 (GND), U17.2, U17.2 (GND); no longer C11.2, C14.2, C16.2, C18.2, C19.2, C21.2, C40.2, C41.2, C56.2, C57.2, R53.1, R9.1, TP26.1, TP3.1, U12.4 (V-), U12.5 (LATCH), U13.4 (V-), U13.5 (LATCH), U2.4 (V-), U4.4 (V-), U5.4 (V-), U6.4 (V-), U7.4 (V-), U8.4 (V-)
- net MODULATED_L: now also D13.1, R68.2; no longer R58.1
- net MODULATED_R: now also D11.1, R66.2; no longer R56.1
- net OUT_L: now also J6.1 (Pin_1); no longer TP25.1
- net OUT_R: now also J5.1 (Pin_1); no longer TP24.1
- net SW_NODE_L: now also C63.2, U15.5 (HS); no longer C48.1
- net SW_NODE_R: no longer C63.2, R54.1, U15.5 (HS)
- net TRIANGLE_WAVE: now also C25.2, R12.1
- net VOL_ADJ_L: now also U7.7; no longer U6.1
- net V_BIAS_L: now also R54.2, U7.6 (-), U8.5 (+), R12.2, R6.2; no longer U6.3 (+), U8.3 (+)
- net V_BIAS_R: now also R53.2, U6.2 (-), U8.3 (+); no longer U3.3 (+), U7.5 (+), U8.5 (+)
- net ~{MODULATED_L}: now also D12.2, R67.2; no longer R57.1
- net ~{MODULATED_R}: now also D10.2, R65.2; no longer R55.1
- net at C42.1, R34.1, R36.2: now also U8.2 (-); no longer U8.6 (-)
- net at U5.5 (+): now also R11.5
- net at U4.5 (+): now also C5.2, R6.1; no longer R5.1
- net at R11.6, R19.1, U6.7: now also R17.2; no longer R15.2
- net at R10.1, TP10.1, U9.1: now also C25.1
- net at R10.2, U9.4 (-): now also R9.1; no longer R9.2
- net at C75.1, C79.1, L8.2: now also R78.2
- net at U14.4 (HOL): now also R73.1
- net at U14.9 (LOL): now also R74.1
- net at R11.3, R18.1: now also R16.2, U6.1; no longer R14.2, U7.7
- net at R19.2, R21.1: now also U7.5 (+); no longer U6.2 (-)
- net at U15.4 (HOL): now also R75.1
- net at C43.1, R35.1, R37.2: now also U8.6 (-); no longer U8.2 (-)
- net at U5.3 (+): now also R11.2; no longer R11.5
- net at U5.1, U5.2 (-): now also R14.1; no longer R17.1
- net at C72.1, C78.1, L7.2: now also R77.2
- net at U15.9 (LOL): now also R76.1
- net at U4.3 (+): now also R5.1, C4.2; no longer R11.2
- new net: C46.1, R49.2
- new net: R15.1, U5.6 (-), U5.7
- new net: C44.1, D4.1 (K), L5.1, R38.2, R40.1
- new net: D4.2 (A), L3.1, U11.2 (Lx1)
- new net: R15.2, R17.1, U6.6 (-)
- new net: FL1.3, J1.2 (Pin_2), TP3.1
- new net: C67.1, D13.3, R68.1, U17.3
- new net: D7.1 (K), R52.1
- new net: D5.1 (K), L4.2, U11.3 (Lx2)
- new net: C45.1, D5.2 (A), L6.1, R39.2, R41.1, U11.4 (VoutN)
- new net: C41.2, R41.2, R48.1, U11.6 (Vfb2)
- new net: C50.2, J4.R, R53.1, TP17.1, U12.2 (+)
- new net: C51.2, J4.T, R54.1, TP18.1, U13.2 (+)
- new net: C40.1, R38.1
- new net: D6.1 (K), R51.1
- new net: C52.1, C54.2, D8.2 (A), R71.2, U14.1 (VDD)
- new net: R14.2, R16.1, U6.3 (+)
- new net: D3.1 (K), R23.1
- new net: R7.1, R8.2, R9.2
- new net: C64.1, D10.3, R65.1, U16.1
- new net: D2.1 (K), R13.1
- new net: D1.1 (K), J1.1 (Pin_1), K1.5, K1.6, R3.2, TP2.1
- new net: D1.2 (A), JP1.1 (A), K1.1
- new net: C2.1, FL1.2, L1.1
- new net: C40.2, R40.2, R47.2, U11.9 (Vfb1)
- new net: C39.1, R48.2, U11.7 (Vref)
- new net: C41.1, R39.1
- new net: C66.1, D12.3, R67.1, U17.1
- new net: C47.1, R50.2
- new net: FL1.1, K1.3, R3.1
- new net: C65.1, D11.3, R66.1, U16.3
- new net: C53.1, C55.2, D9.2 (A), R72.2, U15.1 (VDD)
- new net: R69.1, R70.2, U3.3 (+)
- new net +5V6: C11.1, C14.1, C16.1, C18.1, C19.1, C21.1, C48.1, C56.1, C57.1, D6.2 (A), L5.2, R49.1, TP15.1, U12.1 (V+), U13.1 (V+), U2.8 (V+), U4.8 (V+), U5.8 (V+), U6.8 (V+), U7.8 (V+), U8.8 (V+)
- new net -5V6: C11.2, C14.2, C16.2, C18.2, C19.2, C21.2, C49.1, C56.2, C57.2, L6.2, R50.1, R52.2, TP16.1, U12.4 (V-), U12.5 (LATCH), U13.4 (V-), U13.5 (LATCH), U2.4 (V-), U4.4 (V-), U5.4 (V-), U6.4 (V-), U7.4 (V-), U8.4 (V-)
- new net MODULATED_L_DT: R58.1, TP25.1, U17.6
- new net MODULATED_R_DT: R56.1, TP23.1, U16.6
- new net VCC: U16.5, U16.5 (VCC), U17.5, U17.5 (VCC)
- new net ~{MODULATED_L_DT}: R57.1, TP26.1, U17.4
- new net ~{MODULATED_R_DT}: R55.1, TP24.1, U16.4
- no-connect marks 2 -> 7
Other:
- note added: "1400Khz 1.5A boost & inverting IC with soft-start, 80% eff, trise"
- note added: "20uF MLCC included as local cap for each half bridge on board rear side, 1uF 0402 on board front"
- note added: "24V bus input"
- note added: "2x 1500uF 20% 35VDC AlElec, 2A @ 120Hz"
- note added: "300mA 5V fixed output 80% eff 32C Trise Buck in fixed PWM mode at 500Khz"
- note added: "60uF 50V X7R MLCC, derates to 12uF at 25V"
- note added: "666K triangle wave gen circuitry"
- note added: "Ill throw some tvs diodes for esd / surge? add zener for OV & reverse proection?"
- note added: "Manual 10A relay based softstart for testing, charge time (5*tao) is 2.5s"
- note added: "Pi Filter f3db @5Khz"
- note added: "deadtime gen stage"
- note added: "deadtime set to 14nS (3*tao of RC) RC only applies to PWM falling edges"
- note added: "experiment with different cap values for C68 and C69 (different filter cutoff frequencies, and 1st->2nd stage filter stability)"
- note added: "latch pin on LT1394 grounded or tied to -5V6"
- note added: "max gain 5x, adjust as needed"
- note added: "point of concern -> psrr through to output signal on 24V bus. -> bus has 2810uF of cap, CMC, and pi filter, but no prereg"
- note removed: "20uF MLCC included as local cap for each half bridge, DNP RC snubbers included for each FET"
- note removed: "2V5 shunt refence, resistor sized to allow up to 11.5mA to 2V5 load"
- note removed: "300mA 5V fixed output 80% eff 32C Trise Buck"
- note removed: "50uF 50V X7R MLCC, derates to 10uF at 25V"
- note removed: "Ill throw some tvs diodes for esd / surge? add zener for OV & reverse proection? include soft start circuitry? Connector Selection? Do we want more cap?"
- note removed: "bus cap"
- note removed: "triangle wave gen circuitry"
- company: Adi R -> Adi Ramachandran
- title: class D GaN Amp -> Class-D GaN Audio Amplifier 
- moved on the sheet: C10, C13, C15, C17, C20, C22, C23, C24, C26, C27, C29, C30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

Commit message: shipped rev0 hardware
Parts:
- added C76, C77, C83, C84, C85, C86: .1uF, Capacitor_SMD:C_0603_1608Metric, symbol Device:C_Small
- added C87, C88: .1uF, Capacitor_SMD:C_0402_1005Metric, symbol Device:C_Small
- added R79, R80, R81, R82, R83, R84: 0, Resistor_SMD:R_0603_1608Metric, symbol Device:R
- C11, C14, C16, C18, C19, C21: footprint Capacitor_SMD:C_0402_1005Metric -> Capacitor_SMD:C_0603_1608Metric
Connections:
- net +5V6: now also R79.2, R80.2, R81.2, R82.2, R83.2, R84.2; no longer C11.1, C14.1, C16.1, C18.1, C19.1, C21.1, U2.8 (V+), U4.8 (V+), U5.8 (V+), U6.8 (V+), U7.8 (V+), U8.8 (V+)
- net -5V6: now also C76.2, C77.2, C83.2, C84.2, C85.2, C86.2, C87.1, C88.1; no longer C11.2, C14.2, C16.2, C18.2, C19.2, C21.2, C56.2, C57.2
- net GND: now also C11.2, C14.2, C16.2, C18.2, C19.2, C21.2, C56.2, C57.2, U1.4 (-), C76.1, C77.1, C83.1, C84.1, C85.1, C86.1, C87.2, C88.2
- net V_BIAS_L: no longer U1.4 (-)
- new net: C14.1, R82.1, U5.8 (V+)
- new net: C19.1, R79.1, U2.8 (V+)
- new net: C18.1, R81.1, U6.8 (V+)
- new net: C16.1, R84.1, U8.8 (V+)
- new net: C11.1, R83.1, U4.8 (V+)
- new net: C21.1, R80.1, U7.8 (V+)
Other:
- note added: "added 0 ohm resistors in case of switching noise on input rail"
- moved on the sheet: C11, C14, C16, C18, C19, C21, U2C, U4C, U5C, U6C, U7C, U8C
